Commit message: Added tracked_multi_description

File: base_link_description/urdf/base_link.xacro (robot description, xacro)
@@ -549,5 +549,5 @@
   <parent link="right_back_glide_wheel_holder_v2_1"/>
   <child link="right_glide_wheel_1_v2_1"/>
-  <axis xyz="1.0 0.0 0.0"/>
+  <axis xyz="-1.0 0.0 0.0"/>
 </joint>
 <joint name="Revolute 19" type="continuous">
@@ -555,5 +555,5 @@
   <parent link="right_back_glide_wheel_holder_v2_1"/>
   <child link="right_glide_wheel_2_v2_1"/>
-  <axis xyz="1.0 0.0 0.0"/>
+  <axis xyz="-1.0 0.0 0.0"/>
 </joint>
 <joint name="Revolute 20" type="continuous">
@@ -561,5 +561,5 @@
   <parent link="right_front_glide_wheel_holder_v2_1"/>
   <child link="right_glide_wheel_3_v2_1"/>
-  <axis xyz="1.0 0.0 0.0"/>
+  <axis xyz="-1.0 0.0 0.0"/>
 </joint>
 <joint name="Revolute 21" type="continuous">
@@ -567,5 +567,5 @@
   <parent link="right_front_glide_wheel_holder_v2_1"/>
   <child link="right_glide_wheel_4_v2_1"/>
-  <axis xyz="1.0 0.0 0.0"/>
+  <axis xyz="-1.0 0.0 0.0"/>
 </joint>
 <joint name="Revolute 22" type="continuous">
